File: Hardware/Qwiic Solid State Relay.brd (EAGLE design)
At the start: 185.4 x 91.4 mm, 79 parts, among them J2 Qwiic Right Angle, J3 Qwiic Right Angle, J9 AVR_SPI_PROG_3X2TESTPOINTS, K1 Solid State Relay - 40A, K2 Solid State Relay - 40A, K3 Solid State Relay - 40A, K4 Solid State Relay - 40A, Q1 600mA/40V, Q2 600mA/40V, Q3 600mA/40V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

Commit message: switching pin labels around to match SSR
Connections:
- net 3.3V: now also K1.3, K2.3, K3.3, K4.3; no longer K1.2, K2.2, K3.2, K4.2
- net N$10: now also K2.4; no longer K2.1
- net N$11: now also K4.4; no longer K4.1
- net N$3: now also K1.4; no longer K1.1
- net N$6: now also K3.4; no longer K3.1
Changed lines of the file:
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@@
 <contactref element="J9" pad="2"/>
 <contactref element="R1" pad="2"/>
-<contactref element="K2" pad="2"/>
+<contactref element="K2" pad="3"/>
 <contactref element="R4" pad="2"/>
-<contactref element="K1" pad="2"/>
+<contactref element="K1" pad="3"/>
 <contactref element="R7" pad="2"/>
-<contactref element="K3" pad="2"/>
+<contactref element="K3" pad="3"/>
 <contactref element="R10" pad="2"/>
-<contactref element="K4" pad="2"/>
+<contactref element="K4" pad="3"/>
 <contactref element="D11" pad="A"/>
 <wire x1="58.42" y1="20.74" x2="59.27" y2="21.59" width="0.2032" layer="1"/>
@@
 <signal name="N$10">
 <contactref element="R2" pad="2"/>
-<contactref element="K2" pad="1"/>
+<contactref element="K2" pad="4"/>
 <wire x1="154.94" y1="22.44" x2="156.63" y2="22.44" width="0.2032" layer="1"/>
 <wire x1="158.115" y1="20.955" x2="159.385" y2="20.955" width="0.2032" layer="1"/>
@@
 <signal name="N$3">
 <contactref element="R5" pad="2"/>
-<contactref element="K1" pad="1"/>
+<contactref element="K1" pad="4"/>
 <wire x1="109.22" y1="22.44" x2="110.91" y2="22.44" width="0.2032" layer="1"/>
 <wire x1="112.395" y1="20.955" x2="113.665" y2="20.955" width="0.2032" layer="1"/>
@@
 <signal name="N$6">
 <contactref element="R8" pad="2"/>
-<contactref element="K3" pad="1"/>
+<contactref element="K3" pad="4"/>
 <wire x1="63.5" y1="22.44" x2="65.063" y2="22.44" width="0.2032" layer="1"/>
 <wire x1="66.548" y1="20.955" x2="67.945" y2="20.955" width="0.2032" layer="1"/>
@@
 <signal name="N$11">
 <contactref element="R12" pad="2"/>
-<contactref element="K4" pad="1"/>
+<contactref element="K4" pad="4"/>
 <wire x1="17.78" y1="22.44" x2="18.962" y2="22.44" width="0.2032" layer="1"/>
 <wire x1="20.447" y1="20.955" x2="22.225" y2="20.955" width="0.2032" layer="1"/>
